Commit message: can say successful in two case

File: urdf_description/robot_description/ridgeback_dual_arm_description/urdf/vkc_big_task.urdf.xacro (robot description, xacro)
@@ -67,8 +67,9 @@
     <parent link="world"/>
     <child link="dynamic_pedestrian"/>
-    <origin xyz="0.6 4.5 1.5" rpy="0 0 0" />
+    <origin xyz="-0.1 4.5 1.5" rpy="0 0 0" />
     <axis xyz="0 1 0"/>
     <limit effort="20" velocity="0.5" lower="-6" upper="6"/>
   </joint>
+  <!-- pervious is 0.6 -->
   <!-- ridgeback robot end -->
 </robot>
