Commit message: final commit, project end

File: urdf_description/robot_description/ridgeback_dual_arm_description/urdf/ridgeback_dual_arm.urdf.xacro (robot description, xacro)
@@ -87,6 +87,6 @@
       </material>
     </visual>
-  </link>
-  <joint name="left_gripper_flange_joint" type="fixed">
+  </link> -->
+  <!-- <joint name="left_gripper_flange_joint" type="fixed">
     <origin xyz="0 0 0" rpy="0 0 0" />
     <parent link="left_arm_tool0" />

File: urdf_description/robot_description/ridgeback_dual_arm_description/urdf/vkc_big_task.urdf.xacro (robot description, xacro)
@@ -4,5 +4,6 @@
   <xacro:include filename="$(find ridgeback_dual_arm_description)/urdf/ridgeback_dual_arm.urdf.xacro" /> <!-- 内部修改 -->
   <!-- scence urdf living room -->
-  <xacro:include filename="$(find env_description)/livingroom_env/main_fixed.xacro"/> <!-- 外部修改 -->
+  <!-- <xacro:include filename="$(find env_description)/livingroom_env/main_fixed.xacro"/> 外部修改 -->
+  <link name = "world"/>
   <!-- Arguments -->
   <xacro:arg name="base_loc_x" default="0.0"/>
