Commit message: pick exp only one left

File: urdf_description/env_description/livingroom_env/main_revolute_door.xacro (robot description, xacro)
@@ -46,4 +46,7 @@
         <box size="0.2 11.1 2" />
       </geometry>
+      <material name="custom_color">
+        <color rgba="0.943 0.765 0.461 1" />
+      </material>
     </visual>
     <collision>
@@ -66,4 +69,7 @@
         <box size="0.2 5 2" />
       </geometry>
+      <material name="custom_color">
+        <color rgba="0.943 0.765 0.461 1" />
+      </material>
     </visual>
     <collision>
@@ -106,4 +112,7 @@
         <box size="0.2 5 2" />
       </geometry>
+      <material name="custom_color">
+        <color rgba="0.943 0.765 0.461 1" />
+      </material>
     </visual>
     <collision>

File: urdf_description/robot_description/ridgeback_dual_arm_description/urdf/vkc_big_task.urdf.xacro (robot description, xacro)
@@ -64,5 +64,5 @@
     </collision>
   </link>
-  <joint name="dynamic_pedestrian_joint" type="prismatic">
+  <!-- <joint name="dynamic_pedestrian_joint" type="prismatic">
     <parent link="world"/>
     <child link="dynamic_pedestrian"/>
@@ -70,4 +70,19 @@
     <axis xyz="0 1 0"/>
     <limit effort="20" velocity="0.5" lower="-6" upper="6"/>
+  </joint> -->
+  <joint name="dynamic_pedestrian_joint_y" type="prismatic">
+    <parent link="dynamic_pedestrian_world_x"/>
+    <child link="dynamic_pedestrian"/>
+    <origin xyz="0.0 0.0 1.5" rpy="0 0 0" />
+    <axis xyz="0 1 0"/>
+    <limit effort="20" velocity="0.3" lower="-8" upper="0.5"/>
+  </joint>
+  <link name ="dynamic_pedestrian_world_x"/>
+  <joint name="dynamic_pedestrian_joint_x" type="prismatic">
+    <parent link="world"/>
+    <child link="dynamic_pedestrian_world_x"/>
+    <origin xyz="-0.1 4.5 0.0" rpy="0 0 0" />
+    <axis xyz="1 0 0"/>
+    <limit effort="20" velocity="0.3" lower="-3" upper="2"/>
   </joint>
   <!-- pervious is 0.6 -->
