Commit message: mpc data process

File: urdf_description/env_description/livingroom_env/main_fixed.xacro (robot description, xacro)
@@ -46,4 +46,7 @@
         <box size="0.2 11.1 2" />
       </geometry>
+      <material name="custom_color">
+        <color rgba="0.943 0.765 0.461 1" />
+      </material>
     </visual>
     <collision>
@@ -66,4 +69,7 @@
         <box size="0.2 5 2" />
       </geometry>
+      <material name="custom_color">
+        <color rgba="0.943 0.765 0.461 1" />
+      </material>
     </visual>
     <collision>
@@ -106,4 +112,7 @@
         <box size="0.2 5 2" />
       </geometry>
+      <material name="custom_color">
+        <color rgba="0.943 0.765 0.461 1" />
+      </material>
     </visual>
     <collision>
